Commit message: Merge! Enhance simulation configuration and control integration
- Update VSCode settings for ROS2 workspace directory.
- Adjust URDF for robot base positioning in the simulation environment.
- Modify camera simulation parameters for improved alignment.
- Add camera marker functionality in the simulation node for better visualization.
- Refactor launch files to include new trajectory topic and robot description generation.
- Introduce simulation controllers configuration for joint trajectory control.
- Add CLAUDE.md for project guidance and documentation.

File: ros2_ws/src/holo_assist_depth_tracker/worlds/urdf/holoassist_scene.urdf.xacro (robot description, xacro)
@@ -151,8 +151,12 @@
     </collision>
   </link>
+  <!-- Robot base in workspace_frame coords:
+       board left edge=0, right=0.700  → robot at x=0.450 → board-centre x=0.450-0.350=+0.100
+       board front edge=0, back=0.500 → robot at y=0.564 → board-centre y=0.564-0.250=+0.314
+       Robot base joint is 15 mm below board surface (z=-0.015). -->
   <joint name="workspace_to_ur3e_base" type="fixed">
     <parent link="workspace_frame"/>
     <child link="ur3e_base_link0"/>
-    <origin xyz="0.000 0.314 -0.015" rpy="0 0 0"/>
+    <origin xyz="0.100 0.314 -0.015" rpy="0 0 0"/>
   </joint>
   <xacro:if value="$(arg enable_camera)">
