Commit message: Refactor and enhance robot control and simulation configuration
- Updated perception nodes to handle NumPy float compatibility for Ubuntu 22.04.
- Changed fixed frame from `base_link` to `world` in RViz configuration files.
- Adjusted workspace frame transformations to use `world` as the parent frame.
- Introduced a new configuration file for URSim with appropriate parameters.
- Added joint state topic handling in the coordinate listener and moveit control node.
- Enhanced pick and place sequencer to support home position movements before and after actions.
- Updated launch files to include new parameters for joint state and robot base yaw.
- Improved error handling and state management in the moveit control node for joint goals.
- Refactored perception stack launch to use GroupAction for better organization.

File: ros2_ws/src/ur_onrobot/ur_onrobot_description/urdf/ur_onrobot_macro.xacro (robot description, xacro)
@@ -37,5 +37,5 @@
             input_recipe_filename="${input_recipe_filename}"
         >
-            <origin xyz="0 0 0" rpy="0 0 0" />
+            <xacro:insert_block name="origin" />
         </xacro:ur_robot>
         <!--Create the OnRobot model -->
